File: Electonics/Robot Base/Processor.sch (KiCad schematic (older format))
At the start: 44 parts, among them J1 Conn_01x05_Shielded, J2 SlimStack 0.8mm 2x20, J3 Tag Connect, SW1 SW_Push, U1 STM32F401VCT6, Y1 25MHz

Commit message: Corrected part information for USB
Parts:
- J1: Cost 1.47 -> 0.95; Description USB Micro B Socket, RATH -> USB Micro B Socket, RA SM; Manufacturer Part Number 629105150521 -> 65100516121; Supplier Part Number 732-5960-1-ND -> 732-2109-1-ND
Changed lines of the file:
@@
 F 3 "~" H 6900 4500 50  0001 C CNN
 F 4 "USB B Mini" H 7200 4500 50  0000 C CNN "Label"
-F 5 "1.47" H 6900 4500 50  0001 C CNN "Cost"
-F 6 "USB Micro B Socket, RATH" H 6900 4500 50  0001 C CNN "Description"
+F 5 "0.95" H 6900 4500 50  0001 C CNN "Cost"
+F 6 "USB Micro B Socket, RA SM" H 6900 4500 50  0001 C CNN "Description"
 F 7 "Wurth" H 6900 4500 50  0001 C CNN "Manufacturer"
-F 8 "629105150521" H 6900 4500 50  0001 C CNN "Manufacturer Part Number"
+F 8 "65100516121" H 6900 4500 50  0001 C CNN "Manufacturer Part Number"
 F 9 "Digikey" H 6900 4500 50  0001 C CNN "Supplier"
-F 10 "732-5960-1-ND" H 6900 4500 50  0001 C CNN "Supplier Part Number"
+F 10 "732-2109-1-ND" H 6900 4500 50  0001 C CNN "Supplier Part Number"
 	1    6900 4500
 	-1   0    0    -1
