File: Electonics/Rover/Rover.kicad_pcb (KiCad board)
At the start: 2 copper layers, 56 x 56 mm, 50 parts, among them J1 Conn_01x03, J2 SlimStack 0.8mm 2x20, J3 Conn_01x03, Q1 FDV303N, Q2 FDV303N, Q3 FDV303N, Q4 FDV303N, T1 Rover vA, T2 Board ID, T3 Ball Caster, U1 TCRT1000, U2 TPS54202, U3 TCRT1000

Commit message: Minor tidy-up of some of the files.
Added set of instructions for setting up the library paths and BoM generation.
Other:
- rule pad_to_mask_clearance: 0 -> 0.05
